File: RIP_ExtensionBoard/RIP_ExtensionBoard.kicad_pcb (KiCad board)
At the start: 2 copper layers, 200 x 108 mm, 27 parts, among them J1 Power In, J2 MD20A, J3 Theta Encoder, J4 Alpha Encoder, J5 Emergency Logic, J7 HC05, U1 NUCLEO-G474RE, U2 LM317_TO-220

Commit message: fix footprint
Parts:
- J1: footprint Connector_Phoenix_GMSTB:PhoenixContact_GMSTBA_2,5_2-G-7,62_1x02_P7.62mm_Horizontal -> Connector_Phoenix_MC_HighVoltage:PhoenixContact_MC_1,5_2-G-5.08_1x02_P5.08mm_Horizontal
- J2: footprint Connector_Phoenix_GMSTB:PhoenixContact_GMSTBA_2,5_3-G-7,62_1x03_P7.62mm_Horizontal -> Connector_Phoenix_MC_HighVoltage:PhoenixContact_MC_1,5_3-G-5.08_1x03_P5.08mm_Horizontal
- J3, J4, J5: footprint Connector_Phoenix_GMSTB:PhoenixContact_GMSTBA_2,5_4-G-7,62_1x04_P7.62mm_Horizontal -> Connector_Phoenix_MC_HighVoltage:PhoenixContact_MC_1,5_4-G-5.08_1x04_P5.08mm_Horizontal
- moved J1 4.35 mm to (80.2, 53.5)
- moved J2 4.35 mm to (140.8, 53.5)
- moved J3 4.35 mm to (103.0, 53.5)
- moved J4 4.35 mm to (170.9, 53.5)
- moved J5 4.35 mm to (205.5, 53.5)
Routing:
- net Net-(J5-Pin_2): track 37.2 -> 45.2 mm
- net DIR: track 85.4 -> 93.4 mm
- net +3.3V: track 275.4 -> 282.6 mm
- net theta_B: track 88.6 -> 95.4 mm
- net +5V: track 403.6 -> 409.4 mm
- net theta_A: track 96.8 -> 102.6 mm
- net PWM: track 95.4 -> 100.1 mm
- net alpha_A: track 77.1 -> 81.7 mm
- net alpha_B: track 55.2 -> 59.0 mm

Commit message: rewiring
Parts:
- removed H5, H6: MountingHole_Pad, MountingHole:MountingHole_2.2mm_M2_DIN965_Pad
- removed R1: 330, Resistor_THT:R_Axial_DIN0309_L9.0mm_D3.2mm_P12.70mm_Horizontal
- removed R2: 470, Resistor_THT:R_Axial_DIN0309_L9.0mm_D3.2mm_P12.70mm_Horizontal
- removed R3: 75, Resistor_THT:R_Axial_DIN0309_L9.0mm_D3.2mm_P12.70mm_Horizontal
- moved G*** 54.5 mm to (84.1, 68.4)
- moved R4 22.9 mm to (75.2, 67.9)
- moved D1 22.9 mm to (56.3, 67.9)
Connections:
- D2 pad 1: Net-(D2-K) -> Emergency
- R6 pad 1: Net-(D2-K) -> Emergency
- U2 pad 1: Net-(U2-ADJ) -> GND
Routing:
- net GND: track 0.00 -> 526.6 mm
- net +3.3V: track 282.6 -> 226.5 mm, vias 0 -> 1
- net Emergency: track 22.3 -> 58.5 mm
- net Net-(U2-ADJ): track 35.5 -> 0.00 mm
- net +5V: track 409.4 -> 441.1 mm, vias 0 -> 3
- net Net-(D2-K): track 30.5 -> 0.00 mm
- net LCD_RD: track 165.0 -> 137.8 mm
- net LCD_RST: track 140.9 -> 119.3 mm
- net Net-(R2-Pad1): track 20.9 -> 0.00 mm
- net LCD_WR: track 154.5 -> 134.0 mm
- net alpha_A: track 81.7 -> 64.0 mm, vias 0 -> 2
- net LCD_RS: track 141.1 -> 125.1 mm
- net theta_B: track 95.4 -> 109.9 mm, vias 0 -> 2
- net STM_RX: track 115.9 -> 101.8 mm
- net theta_A: track 102.6 -> 116.3 mm, vias 0 -> 2
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- added copper zone on F.Cu, net GND
Other:
- board text added: "LM1117T-3.3"
- board text removed: "330"
- board text removed: "470"
- board text removed: "75"
- board text removed: "LM317"
