File: RIP_STM32G474RET6/RIP_STM32G474RET6.kicad_sch (KiCad schematic)
At the start: 35 parts, among them J1 USB_C_Receptacle_USB2.0_14P, J2 Conn_01x04, J3 Conn_01x03, J4 Conn_01x03, J5 Jack-DC, J6 Screw_Terminal_01x02, SW1 SW_Push, SW2 SW_Push, U1 STM32G474RETx, U2 AMS1117-3.3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

Commit message: rewiring
Parts:
- C1, C10, C11, C12, C13, C14, C15, C2, C3, C4, C5, C6, C7, C8, C9: footprint (none) -> Capacitor_SMD:C_0402_1005Metric
- D1, D2, D3: footprint (none) -> LED_SMD:LED_0603_1608Metric
- J1: footprint (none) -> Connector_USB:USB_C_Receptacle_GCT_USB4105-xx-A_16P_TopMnt_Horizontal
- J2: footprint (none) -> Connector_PinHeader_2.54mm:PinHeader_1x04_P2.54mm_Vertical
- J3, J4: footprint (none) -> Connector_PinHeader_2.54mm:PinHeader_1x03_P2.54mm_Vertical
- J5: footprint (none) -> Connector_BarrelJack:BarrelJack_Horizontal
- J6: footprint (none) -> TerminalBlock_Phoenix:TerminalBlock_Phoenix_MKDS-1,5-2-5.08_1x02_P5.08mm_Horizontal
- R1, R2, R3, R4, R5: footprint (none) -> Resistor_SMD:R_0402_1005Metric
- SW1, SW2: footprint (none) -> Button_Switch_SMD:SW_SPST_PTS810
- Y1, Y2: footprint (none) -> Crystal:Crystal_SMD_MicroCrystal_CC7V-T1A-2Pin_3.2x1.5mm
Connections:
- net PC2: now reaches U1.10 (PC2)
- net PC3: now reaches U1.11 (PC3)
- net PA1: now reaches U1.13 (PA1)
- net PA2: now reaches U1.14 (PA2)
- net PA3: now reaches U1.17 (PA3)
- net PA4: now reaches U1.18 (PA4)
- net PA5: now reaches U1.19 (PA5)
- net PA6: now reaches U1.20 (PA6)
- net PA7: now reaches U1.21 (PA7)
- net PC4: now reaches U1.22 (PC4)
- net PC5: now reaches U1.23 (PC5)
- net PB0: now reaches U1.24 (PB0)
- net PB1: now reaches U1.25 (PB1)
- net PB2: now reaches U1.26 (PB2)
- net PB10: now reaches U1.30 (PB10)
- net PB11: now reaches U1.33 (PB11)
- net PB12: now reaches U1.34 (PB12)
- net PB13: now reaches U1.35 (PB13)
- net PB14: now reaches U1.36 (PB14)
- net PB15: now reaches U1.37 (PB15)
- net PC6: now reaches U1.38 (PC6)
- net PC7: now reaches U1.39 (PC7)
- net PC8: now reaches U1.40 (PC8)
- net PC9: now reaches U1.41 (PC9)
- net PA8: now reaches U1.42 (PA8)
- net PA9: now reaches U1.43 (PA9)
- net PA10: now reaches U1.44 (PA10)
- net PA15: now reaches U1.51 (PA15)
- net PC10: now reaches U1.52 (PC10)
- net PC11: now reaches U1.53 (PC11)
- net PD2: now reaches U1.55 (PD2)
- net PB3: now reaches U1.56 (PB3)
- net PB4: now reaches U1.57 (PB4)
- net PB5: now reaches U1.58 (PB5)
- net PB6: now reaches U1.59 (PB6)
- net PB7: now reaches U1.60 (PB7)
- net PB9: now reaches U1.62 (PB9)
- net PC0: now reaches U1.8 (PC0)
- net PC1: now reaches U1.9 (PC1)
Other:
- moved on the sheet: C1, C10, C11, C12, C13, C14, C15, C2, C3, C4, C5, C6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

Commit message: chip
Parts:
- removed C1, C2, C3, C4: 10pf, Capacitor_SMD:C_0402_1005Metric, symbol Device:C
- removed C10, C11, C5, C8, C9: 100nf, Capacitor_SMD:C_0402_1005Metric, symbol Device:C
- removed C12, C14: 10nf, Capacitor_SMD:C_0402_1005Metric, symbol Device:C
- removed C13, C15: 1uf, Capacitor_SMD:C_0402_1005Metric, symbol Device:C
- removed C6: 10uf, Capacitor_SMD:C_0402_1005Metric, symbol Device:C
- removed C7: 22uf, Capacitor_SMD:C_0402_1005Metric, symbol Device:C
- removed D1: Green LED, LED_SMD:LED_0603_1608Metric, symbol Device:LED
- removed D2: Blue LED, LED_SMD:LED_0603_1608Metric, symbol Device:LED
- removed D3: Red LED, LED_SMD:LED_0603_1608Metric, symbol Device:LED
- removed J1: USB_C_Receptacle_USB2.0_14P, Connector_USB:USB_C_Receptacle_GCT_USB4105-xx-A_16P_TopMnt_Horizontal, symbol Connector:USB_C_Receptacle_USB2.0_14P
- removed J2: Conn_01x04, Connector_PinHeader_2.54mm:PinHeader_1x04_P2.54mm_Vertical, symbol Connector_Generic:Conn_01x04
- removed J3, J4: Conn_01x03, Connector_PinHeader_2.54mm:PinHeader_1x03_P2.54mm_Vertical, symbol Connector_Generic:Conn_01x03
- removed J5: Jack-DC, Connector_BarrelJack:BarrelJack_Horizontal, symbol Connector:Jack-DC
- removed J6: Screw_Terminal_01x02, TerminalBlock_Phoenix:TerminalBlock_Phoenix_MKDS-1,5-2-5.08_1x02_P5.08mm_Horizontal, symbol Connector:Screw_Terminal_01x02
- removed R2: 5.1k, Resistor_SMD:R_0402_1005Metric, symbol Device:R
- removed R3, R4: 100, Resistor_SMD:R_0402_1005Metric, symbol Device:R
- removed SW1, SW2: SW_Push, Button_Switch_SMD:SW_SPST_PTS810, symbol Switch:SW_Push
- removed U1: STM32G474RETx, Package_QFP:LQFP-64_10x10mm_P0.5mm, symbol MCU_ST_STM32G4:STM32G474RETx
- removed U2: AMS1117-3.3, Package_TO_SOT_SMD:SOT-223-3_TabPin2, symbol Regulator_Linear:AMS1117-3.3
- removed Y1: 8 MHz, Crystal:Crystal_SMD_MicroCrystal_CC7V-T1A-2Pin_3.2x1.5mm, symbol Device:Crystal
- removed Y2: 32.768 Mhz, Crystal:Crystal_SMD_MicroCrystal_CC7V-T1A-2Pin_3.2x1.5mm, symbol Device:Crystal
- added A1: Color Shield, Module:Arduino_UNO_R3, symbol MCU_Module:Arduino_UNO_R3
- added A2: TFT LCD Shield, Module:Arduino_UNO_R3, symbol MCU_Module:Arduino_UNO_R3
- added D2: 1N47xxA, Diode_THT:D_DO-41_SOD81_P10.16mm_Horizontal, symbol Diode:1N47xxA
- added H1, H2, H3, H4: MountingHole, MountingHole:MountingHole_3mm, symbol Mechanical:MountingHole
- added J1: HC05, Connector_PinSocket_2.54mm:PinSocket_1x06_P2.54mm_Vertical, symbol Connector_Generic:Conn_01x06
- added J2: MD20A, Connector_Phoenix_MC_HighVoltage:PhoenixContact_MC_1,5_3-G-5.08_1x03_P5.08mm_Horizontal, symbol Connector:Screw_Terminal_01x03
- added J3: Theta Encoder, Connector_Phoenix_MC_HighVoltage:PhoenixContact_MC_1,5_4-G-5.08_1x04_P5.08mm_Horizontal, symbol Connector:Screw_Terminal_01x04
- added J4: Alpha Encoder, Connector_Phoenix_MC_HighVoltage:PhoenixContact_MC_1,5_4-G-5.08_1x04_P5.08mm_Horizontal, symbol Connector:Screw_Terminal_01x04
- added J5: Emergency Logic, Connector_Phoenix_MC_HighVoltage:PhoenixContact_MC_1,5_4-G-5.08_1x04_P5.08mm_Horizontal, symbol Connector:Screw_Terminal_01x04
- R1: value 5.1k -> 20; footprint Resistor_SMD:R_0402_1005Metric -> Resistor_THT:R_Axial_DIN0309_L9.0mm_D3.2mm_P12.70mm_Horizontal
- R5: value 100 -> 1k; footprint Resistor_SMD:R_0402_1005Metric -> Resistor_THT:R_Axial_DIN0309_L9.0mm_D3.2mm_P12.70mm_Horizontal
Connections:
- net BOOT0 is gone; now on net GND: R5.1
- net +3.3V: now also A2.4 (3V3), J3.1 (Pin_1), J4.1 (Pin_1)
- net +5V: now also A1.5 (+5V), A2.5 (+5V), J1.5 (Pin_5), J5.1 (Pin_1)
- net GND: now also A1.6 (GND), A1.7 (GND), A2.7 (GND), D2.2 (A), J1.4 (Pin_4), J2.3 (Pin_3), J3.4 (Pin_4), J4.4 (Pin_4); no longer R1.2
- net Emergency: now reaches R1.1
- net Emergency: now also D2.1 (K)
- net at R5.2: now also R1.2, J5.2 (Pin_2), J5.3 (Pin_3), J5.4 (Pin_4)
- new net C0: A1.23 (D8)
- new net C1: A1.24 (D9)
- new net C2: A1.25 (D10)
- new net C3: A1.26 (D11)
- new net C4: A1.27 (D12)
- new net C5: A1.28 (D13)
- new net C6: A1.18 (D3)
- new net C7: A1.19 (D4)
- new net DIR: J2.2 (Pin_2)
- new net LAT: A1.10 (A1)
- new net LCD_CS: A2.12 (A3)
- new net LCD_D0: A2.23 (D8)
- new net LCD_D1: A2.24 (D9)
- new net LCD_D2: A2.17 (D2)
- new net LCD_D3: A2.18 (D3)
- new net LCD_D4: A2.19 (D4)
- new net LCD_D5: A2.20 (D5)
- new net LCD_D6: A2.21 (D6)
- new net LCD_D7: A2.22 (D7)
- new net LCD_RD: A2.9 (A0)
- new net LCD_RS: A2.11 (A2)
- new net LCD_RST: A2.13 (SDA/A4)
- new net LCD_WR: A2.10 (A1)
- new net PWM: J2.1 (Pin_1)
- new net RSTn: A1.11 (A2)
- new net SB: A1.9 (A0)
- new net SCK: A1.21 (D6)
- new net SDA: A1.22 (D7)
- new net SD_CS: A2.25 (D10)
- new net SD_DI: A2.26 (D11)
- new net SD_DO: A2.27 (D12)
- new net SD_SCK: A2.28 (D13)
- new net STM_RX: J1.3 (Pin_3)
- new net STM_TX: J1.2 (Pin_2)
- new net alpha_A: J4.2 (Pin_2)
- new net alpha_B: J4.3 (Pin_3)
- new net theta_A: J3.2 (Pin_2)
- new net theta_B: J3.3 (Pin_3)
- no-connect marks 0 -> 28
Other:
- added sheet STM32G474RET6 (STM32G474RET6.kicad_sch)
- note removed: "Clock Management"
- note removed: "Power Management"
- note removed: "Power Supply Scheme"
- note removed: "Uploader"
- title: RIP STM32G474RET6 -> Root
