File: RIP_STM32G474RET6/RIP_STM32G474RET6.kicad_pcb (KiCad board)
At the start: 2 copper layers, 35 parts, among them J1 USB_C_Receptacle_USB2.0_14P, J2 Conn_01x04, J3 Conn_01x03, J4 Conn_01x03, J5 Jack-DC, J6 Screw_Terminal_01x02, SW1 SW_Push, SW2 SW_Push, U1 STM32G474RETx, U2 AMS1117-3.3, Y1 8 MHz, Y2 32.768 Mhz

Commit message: chip
Parts:
- removed C1, C2, C3, C4: 10pf, Capacitor_SMD:C_0402_1005Metric
- removed C10, C11, C5, C8, C9: 100nf, Capacitor_SMD:C_0402_1005Metric
- removed C12, C14: 10nf, Capacitor_SMD:C_0402_1005Metric
- removed C13, C15: 1uf, Capacitor_SMD:C_0402_1005Metric
- removed C6: 10uf, Capacitor_SMD:C_0402_1005Metric
- removed C7: 22uf, Capacitor_SMD:C_0402_1005Metric
- removed D1: Green LED, LED_SMD:LED_0603_1608Metric
- removed D3: Red LED, LED_SMD:LED_0603_1608Metric
- removed R3, R4: 100, Resistor_SMD:R_0402_1005Metric
- removed SW1, SW2: SW_Push, Button_Switch_SMD:SW_SPST_PTS810
- removed U2: AMS1117-3.3, Package_TO_SOT_SMD:SOT-223-3_TabPin2
- removed Y1: 8 MHz, Crystal:Crystal_SMD_MicroCrystal_CC7V-T1A-2Pin_3.2x1.5mm
- removed Y2: 32.768 Mhz, Crystal:Crystal_SMD_MicroCrystal_CC7V-T1A-2Pin_3.2x1.5mm
- added A1: Color Shield, Module:Arduino_UNO_R3, B.Cu at (86.1, 109.0)
- added A2: TFT LCD Shield, Module:Arduino_UNO_R3, B.Cu at (147.8, 109.0)
- added C16: 100nf, Capacitor_SMD:C_0402_1005Metric, F.Cu at (147.9, 56.8)
- added C17: 10nf, Capacitor_SMD:C_0402_1005Metric, F.Cu at (144.7, 71.5)
- added C18: 1uf, Capacitor_SMD:C_0402_1005Metric, F.Cu at (142.8, 71.5)
- added C19: 100nf, Capacitor_SMD:C_0402_1005Metric, F.Cu at (136.4, 52.9)
- added C20: 100nf, Capacitor_SMD:C_0402_1005Metric, F.Cu at (132.4, 64.3)
- added C21: 10nf, Capacitor_SMD:C_0402_1005Metric, F.Cu at (148.6, 71.5)
- added C22: 100nf, Capacitor_SMD:C_0402_1005Metric, F.Cu at (143.9, 68.3)
- added C23: 1uf, Capacitor_SMD:C_0402_1005Metric, F.Cu at (146.7, 71.5)
- added C24: 100nf, Capacitor_SMD:C_0402_1005Metric, F.Cu at (116.0, 53.3)
- added C25: 10uf, Capacitor_SMD:C_0402_1005Metric, F.Cu at (102.7, 49.4)
- added C26: 10pf, Capacitor_SMD:C_0402_1005Metric, F.Cu at (125.2, 52.5)
- added C27: 10pf, Capacitor_SMD:C_0402_1005Metric, F.Cu at (125.2, 58.4)
- added C28: 22uf, Capacitor_SMD:C_0402_1005Metric, F.Cu at (106.3, 49.4)
- added C29: 10pf, Capacitor_SMD:C_0402_1005Metric, F.Cu at (125.2, 62.7)
- added C30: 10pf, Capacitor_SMD:C_0402_1005Metric, F.Cu at (125.2, 68.6)
- added D5: Green LED, LED_SMD:LED_0603_1608Metric, F.Cu at (103.4, 62.0)
- added D6: Blue LED, LED_SMD:LED_0603_1608Metric, F.Cu at (103.4, 66.2)
- added G***: LOGO, LOGO, F.Cu at (155.4, 61.9)
- added H1: MountingHole, MountingHole:MountingHole_3mm, F.Cu at (79.1, 33.8)
- added H2: MountingHole, MountingHole:MountingHole_3mm, F.Cu at (203.0, 33.7)
- added H3: MountingHole, MountingHole:MountingHole_3mm, F.Cu at (79.1, 147.0)
- added H4: MountingHole, MountingHole:MountingHole_3mm, F.Cu at (203.0, 146.9)
- added J10: Conn_01x03, Connector_PinHeader_2.54mm:PinHeader_1x03_P2.54mm_Vertical, F.Cu at (86.5, 52.3)
- added J11: Jack-DC, Connector_BarrelJack:BarrelJack_Horizontal, F.Cu at (90.0, 44.7)
- added J12: Screw_Terminal_01x02, Connector_Phoenix_MC_HighVoltage:PhoenixContact_MC_1,5_2-G-5.08_1x02_P5.08mm_Horizontal, B.Cu at (100.1, 39.2)
- added J7: USB_C_Receptacle_USB2.0_14P, Connector_USB:USB_C_Receptacle_GCT_USB4105-xx-A_16P_TopMnt_Horizontal, F.Cu at (81.1, 69.9)
- added J9: Conn_01x04, Connector_PinHeader_2.54mm:PinHeader_1x04_P2.54mm_Vertical, F.Cu at (94.5, 52.3)
- added R10: 100, Resistor_SMD:R_0402_1005Metric, F.Cu at (106.0, 66.2)
- added R6: 5.1k, Resistor_SMD:R_0402_1005Metric, F.Cu at (88.4, 71.3)
- added R7: 5.1k, Resistor_SMD:R_0402_1005Metric, F.Cu at (88.4, 73.2)
- added R9: 100, Resistor_SMD:R_0402_1005Metric, F.Cu at (106.0, 62.0)
- added SW3: SW_Push, Button_Switch_SMD:SW_SPST_PTS810, F.Cu at (116.0, 64.6)
- added SW4: SW_Push, Button_Switch_SMD:SW_SPST_PTS810, F.Cu at (116.0, 56.9)
- added U3: STM32G474RETx, Package_QFP:LQFP-64_10x10mm_P0.5mm, F.Cu at (140.1, 60.6)
- added U4: AMS1117-3.3, Package_TO_SOT_SMD:SOT-223-3_TabPin2, F.Cu at (104.4, 55.0)
- added Y3: 32.768 Mhz, Crystal:Crystal_SMD_MicroCrystal_CC7V-T1A-2Pin_3.2x1.5mm, F.Cu at (125.2, 55.5)
- added Y4: 8 MHz, Crystal:Crystal_SMD_MicroCrystal_CC7V-T1A-2Pin_3.2x1.5mm, F.Cu at (125.2, 65.6)
- D2: value Blue LED -> 1N47xxA; footprint LED_SMD:LED_0603_1608Metric -> Diode_THT:D_DO-41_SOD81_P10.16mm_Horizontal
- J1: value USB_C_Receptacle_USB2.0_14P -> HC05; footprint Connector_USB:USB_C_Receptacle_GCT_USB4105-xx-A_16P_TopMnt_Horizontal -> Connector_PinSocket_2.54mm:PinSocket_1x06_P2.54mm_Vertical
- J2: value Conn_01x04 -> MD20A; footprint Connector_PinHeader_2.54mm:PinHeader_1x04_P2.54mm_Vertical -> Connector_Phoenix_MC_HighVoltage:PhoenixContact_MC_1,5_3-G-5.08_1x03_P5.08mm_Horizontal; moved to B.Cu
- J3: value Conn_01x03 -> Theta Encoder; footprint Connector_PinHeader_2.54mm:PinHeader_1x03_P2.54mm_Vertical -> Connector_Phoenix_MC_HighVoltage:PhoenixContact_MC_1,5_4-G-5.08_1x04_P5.08mm_Horizontal; moved to B.Cu
- J4: value Conn_01x03 -> Alpha Encoder; footprint Connector_PinHeader_2.54mm:PinHeader_1x03_P2.54mm_Vertical -> Connector_Phoenix_MC_HighVoltage:PhoenixContact_MC_1,5_4-G-5.08_1x04_P5.08mm_Horizontal; moved to B.Cu
- J5: value Jack-DC -> Emergency Logic; footprint Connector_BarrelJack:BarrelJack_Horizontal -> Connector_Phoenix_MC_HighVoltage:PhoenixContact_MC_1,5_4-G-5.08_1x04_P5.08mm_Horizontal; moved to B.Cu
- J6: value Screw_Terminal_01x02 -> Conn_01x03; footprint TerminalBlock_Phoenix:TerminalBlock_Phoenix_MKDS-1,5-2-5.08_1x02_P5.08mm_Horizontal -> Connector_PinHeader_2.54mm:PinHeader_1x03_P2.54mm_Vertical
- R1: value 5.1k -> 20; footprint Resistor_SMD:R_0402_1005Metric -> Resistor_THT:R_Axial_DIN0309_L9.0mm_D3.2mm_P12.70mm_Horizontal
- R2: value 5.1k -> 1k
- R5: value 100 -> 1k; footprint Resistor_SMD:R_0402_1005Metric -> Resistor_THT:R_Axial_DIN0309_L9.0mm_D3.2mm_P12.70mm_Horizontal
- U1: value STM32G474RETx -> USBLC6-2SC6; footprint Package_QFP:LQFP-64_10x10mm_P0.5mm -> Package_TO_SOT_SMD:SOT-23-6
- moved D2 153.7 mm to (180.5, 54.9), turned to 90 degrees
- moved R1 141.4 mm to (183.9, 50.3)
- moved R5 141.1 mm to (183.9, 45.3)
- moved J4 107.3 mm to (155.7, 39.2)
- moved J6 104.7 mm to (78.4, 52.3), turned to 0 degrees
- moved J1 92.9 mm to (195.8, 55.5), turned to 0 degrees
- moved J2 90.4 mm to (113.6, 39.2)
- moved J3 88.4 mm to (132.1, 39.2)
- moved J5 66.7 mm to (179.3, 39.2), turned to 0 degrees
- moved U1 52.5 mm to (89.4, 66.7), turned to 90 degrees
- moved R2 40.8 mm to (79.3, 61.2)
Connections:
- D2 pad 1: VSSA -> Emergency
- D2 pad 2: Net-(D2-A) -> VSSA
- J2 pad 1: VDD -> PWM
- J2 pad 2: SWDIO-JTMS -> DIR
- J2 pad 3: SWCLK-JTCK -> VSSA
- J3 pad 2: BOOT0 -> theta_A
- J3 pad 3: VSSA -> theta_B
- J4 pad 1: VUSB -> VDD
- J4 pad 2: +5V -> alpha_A
- J4 pad 3: VEXT -> alpha_B
- J5 pad 1: VEXT -> +5V
- J5 pad 2: VSSA -> Net-(J5-Pin_2)
- J5 pad 3: (no net) -> Net-(J5-Pin_2)
- J6 pad 1: VEXT -> VDD
- J6 pad 2: VSSA -> BOOT0
- R1 pad 1: Net-(J1-CC1) -> Emergency
- R1 pad 2: VSSA -> Net-(J5-Pin_2)
- R2 pad 1: VSSA -> Net-(J6-Pin_3)
- R2 pad 2: Net-(J1-CC2) -> VSSA
- R5 pad 1: BOOT0 -> VSSA
- R5 pad 2: Net-(D3-A) -> Net-(J5-Pin_2)
- U1 pad 1: VDD -> Net-(J7-D--PadA7)
- U1 pad 2: PC13 -> VSSA
- U1 pad 3: OSC32_IN -> Net-(J7-D+-PadA6)
- U1 pad 4: OSC32_OUT -> USB_PD
- U1 pad 5: OSC_IN -> VUSB
- U1 pad 6: OSC_OUT -> USB_DM
Routing:
- net VSSA: track 0.00 -> 486.3 mm, vias 0 -> 7
- net +5V: track 0.00 -> 308.5 mm, vias 0 -> 2
- net VDD: track 0.00 -> 296.1 mm, vias 0 -> 7
- net LCD_D2: track 0.00 -> 113.1 mm, vias 0 -> 2
- net LCD_D1: track 0.00 -> 110.5 mm, vias 0 -> 2
- net LCD_D3: track 0.00 -> 108.7 mm, vias 0 -> 2
- net LCD_D4: track 0.00 -> 107.2 mm, vias 0 -> 2
- net LCD_D5: track 0.00 -> 105.7 mm, vias 0 -> 2
- net LCD_D6: track 0.00 -> 104.2 mm, vias 0 -> 2
- net LCD_D7: track 0.00 -> 102.9 mm, vias 0 -> 2
- net SD_DO: track 0.00 -> 101.9 mm, vias 0 -> 2
- net LCD_D0: track 0.00 -> 100.1 mm, vias 0 -> 2
- net SD_DI: track 0.00 -> 99.9 mm
- net RSTn: track 0.00 -> 98.2 mm
- net LAT: track 0.00 -> 96.3 mm
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- added copper zone on F.Cu, net VDD
- added copper zone on In2.Cu, net VDD
- added copper zone on B.Cu, net VSSA
- added copper zone on In1.Cu, net VSSA
Other:
- board outline added: 132 x 120 mm
- copper layers 2 -> 4
- board text added: "2.4″ Touch Screen LCD With SD Card Reader"
- board text added: "3.3V Indicator"
- board text added: "5 VDC"
- board text added: "5V"
- board text added: "Alpha Encoder"
- board text added: "B1"
- board text added: "Color Shield v1.1"
- board text added: "Emergency Switch"
- board text added: "GND"
- board text added: "GND BOOT0 VDD"
- board text added: "GND SWCLK SWDIO VDD"
- board text added: "LD2"
- board text added: "MD20A"
- board text added: "Phakin B. 6637 F10"
- board text added: "Power Input"
- board text added: "RX"
- board text added: "Reset"
- board text added: "Rotary Inverted Pendulum"
- board text added: "TX"
- board text added: "Theta Encoder"
- board text added: "VEXT 5V VUSB"

Commit message: final
Parts:
- moved C23 20.6 mm to (132.4, 56.6)
- moved C18 5.25 mm to (148.0, 71.9), turned to 0 degrees
- moved C17 3.37 mm to (148.0, 70.8)
- moved J7 2.74 mm to (78.3, 69.9)
- moved U1 2.74 mm to (86.6, 66.6)
- moved R6 2.74 mm to (85.7, 71.2)
- moved R7 2.74 mm to (85.7, 73.2)
- moved C21 1.64 mm to (148.0, 73.0)
Routing:
- net VDD: track 296.1 -> 165.7 mm
- net VSSA: track 486.3 -> 462.3 mm, vias 7 -> 15
- net USB_PD: track 70.6 -> 73.3 mm
- net USB_DM: track 73.1 -> 75.7 mm
- added copper zone on F.Cu, net VSSA
- removed copper zone on F.Cu, net VDD
