Commit message: fixed tf

File: src/invpendulum_description/urdf/Rotary_Inverted_Pendulum.urdf (robot description, URDF)
Before this commit: robot Rotary Inverted Pendulum, 3 links, 2 joints
Links:
- removed link Arm_Link1
- removed link Pendulum_Link2
- added link Arm_Link, mass 0.215027242047406; collision mesh filename=package://invpendulum_description/meshes/Arm_Link.STL; visual mesh filename=package://invpendulum_description/meshes/Arm_Link.STL
- added link Pendulum_Link, mass 0.011664; collision mesh filename=package://invpendulum_description/meshes/Pendulum_Link.STL; visual mesh filename=package://invpendulum_description/meshes/Pendulum_Link.STL
Joints:
- joint Rev_Arm: child Arm_Link1 -> Arm_Link
- joint Rev_Pendulum: child Pendulum_Link2 -> Pendulum_Link; parent Arm_Link1 -> Arm_Link

File: src/invpendulum_description/urdf/Rotary_Inverted_Pendulum.xacro (robot description, xacro)
@@ -31,5 +31,5 @@
   </link>
   <!-- Arm Link -->
-  <link name="Arm_Link1">
+  <link name="Arm_Link">
     <inertial>
       <origin xyz="0.0191189780582279 -2.13351893908753e-06 0.0126487945771829" rpy="0 0 0"/>
@@ -46,5 +46,5 @@
       <origin xyz="0 0 0" rpy="0 0 0"/>
       <geometry>
-        <mesh filename="package://invpendulum_description/meshes/Arm_Link1.STL"/>
+        <mesh filename="package://invpendulum_description/meshes/Arm_Link.STL"/>
       </geometry>
       <material name="white">
@@ -55,5 +55,5 @@
       <origin xyz="0 0 0" rpy="0 0 0"/>
       <geometry>
-        <mesh filename="package://invpendulum_description/meshes/Arm_Link1.STL"/>
+        <mesh filename="package://invpendulum_description/meshes/Arm_Link.STL"/>
       </geometry>
     </collision>
@@ -63,9 +63,9 @@
     <origin xyz="0.0002 0 0.212" rpy="0 0 0"/>
     <parent link="base_link"/>
-    <child link="Arm_Link1"/>
+    <child link="Arm_Link"/>
     <axis xyz="0 0 1"/>
   </joint>
   <!-- Pendulum Link -->
-  <link name="Pendulum_Link2">
+  <link name="Pendulum_Link">
     <inertial>
       <origin xyz="0.038074 3.9254e-10 0.0081922" rpy="0 0 0"/>
@@ -82,5 +82,5 @@
       <origin xyz="0 0 0" rpy="0 0 0"/>
       <geometry>
-        <mesh filename="package://invpendulum_description/meshes/Pendulum_Link2.STL"/>
+        <mesh filename="package://invpendulum_description/meshes/Pendulum_Link.STL"/>
       </geometry>
       <material name="lightblue">
@@ -91,5 +91,5 @@
       <origin xyz="0 0 0" rpy="0 0 0"/>
       <geometry>
-        <mesh filename="package://invpendulum_description/meshes/Pendulum_Link2.STL"/>
+        <mesh filename="package://invpendulum_description/meshes/Pendulum_Link.STL"/>
       </geometry>
     </collision>
@@ -98,6 +98,6 @@
   <joint name="Rev_Pendulum" type="continuous">
     <origin xyz="0.1215 0 0.0255" rpy="0 ${pi/2} 0"/>
-    <parent link="Arm_Link1"/>
-    <child link="Pendulum_Link2"/>
+    <parent link="Arm_Link"/>
+    <child link="Pendulum_Link"/>
     <axis xyz="0 0 1"/>
   </joint>

Commit message: complete

File: src/invpendulum_description/urdf/Rotary_Inverted_Pendulum.urdf (robot description, URDF)
Before this commit: robot Rotary Inverted Pendulum, 3 links, 2 joints
Links:
- removed link Arm_Link
- removed link Pendulum_Link
- added link arm_link, mass 0.215027242047406; collision mesh filename=package://invpendulum_description/meshes/arm_link.STL; visual mesh filename=package://invpendulum_description/meshes/arm_link.STL
- added link pendulum_link, mass 0.011664; collision mesh filename=package://invpendulum_description/meshes/pendulum_link.STL; visual mesh filename=package://invpendulum_description/meshes/pendulum_link.STL
Joints:
- joint Rev_Arm: child Arm_Link -> arm_link
- joint Rev_Pendulum: child Pendulum_Link -> pendulum_link; parent Arm_Link -> arm_link

File: src/invpendulum_description/urdf/Rotary_Inverted_Pendulum.xacro (robot description, xacro)
@@ -31,5 +31,5 @@
   </link>
   <!-- Arm Link -->
-  <link name="Arm_Link">
+  <link name="arm_link">
     <inertial>
       <origin xyz="0.0191189780582279 -2.13351893908753e-06 0.0126487945771829" rpy="0 0 0"/>
@@ -46,5 +46,5 @@
       <origin xyz="0 0 0" rpy="0 0 0"/>
       <geometry>
-        <mesh filename="package://invpendulum_description/meshes/Arm_Link.STL"/>
+        <mesh filename="package://invpendulum_description/meshes/arm_link.STL"/>
       </geometry>
       <material name="white">
@@ -55,17 +55,17 @@
       <origin xyz="0 0 0" rpy="0 0 0"/>
       <geometry>
-        <mesh filename="package://invpendulum_description/meshes/Arm_Link.STL"/>
+        <mesh filename="package://invpendulum_description/meshes/arm_link.STL"/>
       </geometry>
     </collision>
   </link>
   <!-- Joint between base and arm -->
-  <joint name="Rev_Arm" type="continuous">
+  <joint name="rev_arm" type="continuous">
     <origin xyz="0.0002 0 0.212" rpy="0 0 0"/>
     <parent link="base_link"/>
-    <child link="Arm_Link"/>
+    <child link="arm_link"/>
     <axis xyz="0 0 1"/>
   </joint>
   <!-- Pendulum Link -->
-  <link name="Pendulum_Link">
+  <link name="pendulum_link">
     <inertial>
       <origin xyz="0.038074 3.9254e-10 0.0081922" rpy="0 0 0"/>
@@ -82,5 +82,5 @@
       <origin xyz="0 0 0" rpy="0 0 0"/>
       <geometry>
-        <mesh filename="package://invpendulum_description/meshes/Pendulum_Link.STL"/>
+        <mesh filename="package://invpendulum_description/meshes/pendulum_link.STL"/>
       </geometry>
       <material name="lightblue">
@@ -91,13 +91,13 @@
       <origin xyz="0 0 0" rpy="0 0 0"/>
       <geometry>
-        <mesh filename="package://invpendulum_description/meshes/Pendulum_Link.STL"/>
+        <mesh filename="package://invpendulum_description/meshes/pendulum_link.STL"/>
       </geometry>
     </collision>
   </link>
   <!-- Joint between arm and pendulum -->
-  <joint name="Rev_Pendulum" type="continuous">
+  <joint name="rev_pendulum" type="continuous">
     <origin xyz="0.1215 0 0.0255" rpy="0 ${pi/2} 0"/>
-    <parent link="Arm_Link"/>
-    <child link="Pendulum_Link"/>
+    <parent link="arm_link"/>
+    <child link="pendulum_link"/>
     <axis xyz="0 0 1"/>
   </joint>

Commit message: new

File: src/invpendulum_description/urdf/Rotary_Inverted_Pendulum.urdf (robot description, URDF)
Before this commit: robot Rotary Inverted Pendulum, 3 links, 2 joints
Links:
- added link end_effector
Joints:
- added joint Pendulum_to_EE: type fixed, parent pendulum_link, child end_effector, origin xyz=0.135 0 0.0115 rpy=0 0 0
